File: PCB_Files/Quad_Board.sch (EAGLE design)
At the start: 32 parts, among them IC2 LM317MB, Q1 32.768kHz, Q2 KX-7 48MHz

Commit message: Board Layout Under Progress
Parts:
- removed 12V_PDB: (no value), pinhead:PINHD-1X2
- removed U$2: NAZE32_FC, Naze32_FCBoard:NAZE32_FC
- added LEVEL_TRANSLATOR1, LEVEL_TRANSLATOR_@, LEVEL_TRANSLATOR_@1: (no value), SparkFun-DigitalIC:TXB0104PWRSOIC14
- added NAZE32_PINHEAD: (no value), pinhead:PINHD-1X10
- added R4, R5, R6: (no value), eagle-ltspice:RR2512
- added SJ1, SJ2, SJ3: SOLDERJUMPERNC2, SparkFun-Passives:SOLDERJUMPERNC2
- renumbered JP1 to MOTHERBOPARD_TX
Connections:
- net N$17 renamed P10.5_V
- removed net 12VDC: 12V_PDB.1
- removed net N$13: ULTRA3.2
- removed net N$3: ULTRA1.2
- removed net N$4: 12V_PDB.2
- removed net N$5: ULTRA3.3
- removed net N$6: MSP1.P9.3/TA3.4
- removed net P5.4_IO_J3.29: MSP1.P5.4/A1, ULTRA5.2
- removed net P5.5_IO_J3.30: MSP1.P5.5/A0, ULTRA6.2
- removed net P5.6_PWM_J4.37: MSP1.P5.6/TA2.1/VREF+/VEREF+/C1.7, ULTRA5.3
- removed net P5.7_IO_J2.17: MSP1.P5.7/TA2.2/VREF-/VEREF-/C1.6, ULTRA6.3
- removed net P6.6_CAPTURE_J4.36: MSP1.P6.6/TA2.3/UCB3SIMO/UCB3SDA/C1.1
- removed net P6.7_CAPTURE_J4.35: MSP1.P6.7/TA2.4/UCB3SOMI/UCB3SCL/C1.0
- removed net P9.1: MSP1.P9.1/A16, ULTRA2.2
- new net 3.3V: LEVEL_TRANSLATOR1.VCCA, LEVEL_TRANSLATOR_@.VCCA, LEVEL_TRANSLATOR_@1.VCCA, SJ1.2, SJ2.2, SJ3.2
- new net 5V: LEVEL_TRANSLATOR1.VCCB, LEVEL_TRANSLATOR_@.VCCB, LEVEL_TRANSLATOR_@1.VCCB
- new net N$1: MSP1.P9.1/A16
- new net N$19: MSP1.P5.4/A1
- new net N$20: MSP1.P5.5/A0
- new net N$25: MSP1.P10.4/TA3.0/C0.7
- new net N$26: MSP1.P10.5/TA3.1/C0.6
- new net OE: LEVEL_TRANSLATOR1.OE, LEVEL_TRANSLATOR_@.OE, LEVEL_TRANSLATOR_@1.OE, R4.2, R5.2, R6.2, SJ1.1, SJ2.1, SJ3.1
- new net P10.3_GPIO5V: LEVEL_TRANSLATOR_@.B4, ULTRA4.3
- new net P10.4_5V: LEVEL_TRANSLATOR_@.B2, ULTRA3.3
- new net P10.5_5V: LEVEL_TRANSLATOR_@.B3
- new net P5.6: LEVEL_TRANSLATOR_@1.A1, MSP1.P5.6/TA2.1/VREF+/VEREF+/C1.7
- new net P5.6_5V: LEVEL_TRANSLATOR_@1.B1, ULTRA5.3
- new net P5.7: LEVEL_TRANSLATOR_@1.A2
- new net P5.7_5V: LEVEL_TRANSLATOR_@1.B2, ULTRA5.2
- new net P6.6: LEVEL_TRANSLATOR_@1.A3, MSP1.P6.6/TA2.3/UCB3SIMO/UCB3SDA/C1.1
- new net P6.6_5V: LEVEL_TRANSLATOR_@1.B3, ULTRA6.3
- new net P6.7: LEVEL_TRANSLATOR_@1.A4, MSP1.P6.7/TA2.4/UCB3SOMI/UCB3SCL/C1.0
- new net P6.7_5V: LEVEL_TRANSLATOR_@1.B4, ULTRA6.2
- new net P8.0_5V: LEVEL_TRANSLATOR1.B1, ULTRA1.2
- new net P8.1_5V: LEVEL_TRANSLATOR1.B2, ULTRA1.3
- new net P8.2_5V: LEVEL_TRANSLATOR1.B3
- new net P8.3_5V: ULTRA2.2
- new net P9.2_5V: LEVEL_TRANSLATOR1.B4, ULTRA2.3
- new net P9.3: LEVEL_TRANSLATOR_@.A1, MSP1.P9.3/TA3.4
- new net P9.3_5V: LEVEL_TRANSLATOR_@.B1, ULTRA3.2
- net 5VDC: now also NAZE32_PINHEAD.2; no longer U$2.5V
- net GND: now also LEVEL_TRANSLATOR1.GND, LEVEL_TRANSLATOR_@.GND, LEVEL_TRANSLATOR_@1.GND, NAZE32_PINHEAD.1, R4.1, R5.1, R6.1; no longer U$2.GND
- net P10.3: now also LEVEL_TRANSLATOR_@.A4
- net P10.4: now also LEVEL_TRANSLATOR_@.A2; no longer MSP1.P10.4/TA3.0/C0.7
- net P10.5: now also LEVEL_TRANSLATOR_@.A3; no longer MSP1.P10.5/TA3.1/C0.6, ULTRA4.3
- net P2.4_PWM_J4.38: now also NAZE32_PINHEAD.10; no longer U$2.8
- net P2.5_PWM_J2.19: now also NAZE32_PINHEAD.9; no longer U$2.7
- net P2.6_PWM_J4.39: now also NAZE32_PINHEAD.8; no longer U$2.6
- net P2.7_PWM_J4.40: no longer U$2.LED/5
- net P3.3_UTXD_J1.4: now also MOTHERBOPARD_TX.1
- net P7.4: now also NAZE32_PINHEAD.6; no longer U$2.U2RX/4
- net P7.5: now also NAZE32_PINHEAD.5; no longer U$2.U2TX/3
- net P7.6: now also NAZE32_PINHEAD.4; no longer U$2.2
- net P7.7: now also NAZE32_PINHEAD.3; no longer U$2.PPM
- net P8.0: now also LEVEL_TRANSLATOR1.A1
- net P8.1: now also LEVEL_TRANSLATOR1.A2, LEVEL_TRANSLATOR1.A3
- net P8.2: no longer ULTRA1.3
- net P9.2: now also LEVEL_TRANSLATOR1.A4; no longer ULTRA2.3
Other:
- note added: "A side Vcc from 1.2 to 3.6V"
- note added: "B side Vcc from 1.65 to 5V"
- note added: "VccA *must* be less than VccB!"

Commit message: Board Layout in Routing Stage
Parts:
- removed SJ1, SJ2, SJ3: SOLDERJUMPERNC2, SparkFun-Passives:SOLDERJUMPERNC2
- added 12V_PDB, MOTHERBOARD_POWER_PINS: (no value), pinhead:PINHD-1X2
- added C14: 680u, rcl:C-EUCM0402
- added C15: 220u, rcl:C-EUCM0402
- added D1: PD3S160, diode:PD3S160
- added L2: 33u, resistor:L-USL2012C
- added LM2596S: LM2596S, national-semiconductor:LM2596S
Connections:
- removed net N$25: MSP1.P10.4/TA3.0/C0.7
- removed net N$26: MSP1.P10.5/TA3.1/C0.6
- removed net OE: LEVEL_TRANSLATOR1.OE, LEVEL_TRANSLATOR_@.OE, LEVEL_TRANSLATOR_@1.OE, R4.2, R5.2, R6.2, SJ1.1, SJ2.1, SJ3.1
- removed net P8.3_5V: ULTRA2.2
- new net 12VDC: 12V_PDB.1, C1.1, C14.1, IC2.IN, LM2596S.VIN
- new net MOTHEROARD_V+: C15.1, L2.2, LM2596S.FB, MOTHERBOARD_POWER_PINS.1
- new net N$10: MSP1.P3.2/PM_UCA2RXD/PM_UCA2SOMI
- new net N$4: D1.C, L2.1, LM2596S.OUT
- net 3.3V: now also LEVEL_TRANSLATOR1.OE, LEVEL_TRANSLATOR_@.OE, LEVEL_TRANSLATOR_@1.OE, R4.2, R5.2, R6.2; no longer SJ1.2, SJ2.2, SJ3.2
- net 5VDC: now also 5V_PDB.1; no longer C1.1, IC2.IN
- net GND: now also 12V_PDB.2, C14.2, C15.2, D1.A, LM2596S.!ON!/OFF, LM2596S.GND, MOTHERBOARD_POWER_PINS.2
- net P10.4: now also MSP1.P10.4/TA3.0/C0.7
- net P10.5: now also MSP1.P10.5/TA3.1/C0.6
- net P2.7_PWM_J4.40: now also NAZE32_PINHEAD.7
- net P5.7: now also MSP1.P5.7/TA2.2/VREF-/VEREF-/C1.6
- net P8.2_5V: now also ULTRA2.2
Other:
- note added: "Level Translators ICs for Ultrasonic Sensors"
- note added: "MotherBoard Power Circuit (5V,2.5A)"
- note added: "Power Suppply Regulation"
- moved on the sheet: 5V_PDB, C1, C10, C11, C12, C13, C2, C3, C4, C5, C6, C7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

Commit message: PCB Layout Rev1 90% done
Parts:
- added R7: (no value), rcl:R-US_0204/5
- added U$1: TXS0102, TXS0102-bi-directional-translator:TXS0102
- renumbered LEVEL_TRANSLATOR_@ to LEVEL_TRANSLATOR_2, LEVEL_TRANSLATOR_@1 to LEVEL_TRANSLATOR_3
Connections:
- removed net N$10: MSP1.P3.2/PM_UCA2RXD/PM_UCA2SOMI
- removed net N$3: MOTHERBOPARD_TX.2
- removed net P3.3_UTXD_J1.4: MOTHERBOPARD_TX.1, MSP1.P3.3/PM_UCA2TXD/PM_UCA2SIMO
- new net A1: MSP1.P3.3/PM_UCA2TXD/PM_UCA2SIMO, U$1.P$5
- new net A2: MOTHERBOPARD_TX.1, U$1.P$4
- new net B1: MSP1.P3.2/PM_UCA2RXD/PM_UCA2SOMI, U$1.P$8
- new net B2: MOTHERBOPARD_TX.2, U$1.P$1
- new net OE: R7.1, U$1.P$6
- net 3V3: now also U$1.P$7
- net 5V: now also U$1.P$3
- net GND: now also R7.2, U$1.P$2

Commit message: MCU Icaps routing remaining
Connections:
- removed net N$19: MSP1.P5.4/A1
- removed net N$20: MSP1.P5.5/A0
- removed net P1.0_LED1: MSP1.P1.0/UCA0STE
- removed net P1.1_BUTTON1: MSP1.P1.1/UCA0CLK
- removed net P1.2_BCLUART_RXD: MSP1.P1.2/UCA0RXD/UCA0SOMI
- removed net P1.3_BCLUART_TXD: MSP1.P1.3/UCA0TXD/UCA0SIMO
- removed net P1.4_BUTTON2: MSP1.P1.4/UCB0STE
- removed net P1.5_SPICLK_J1.7: MSP1.P1.5/UCB0CLK
- removed net P1.6_SPIMOSI_J2.15: MSP1.P1.6/UCB0SIMO/UCB0SDA
- removed net P1.7_SPIMISO_J2.14: MSP1.P1.7/UCB0SOMI/UCB0SCL
- removed net P2.0_RGBLED_RED: MSP1.P2.0/PM_UCA1STE
- removed net P2.1_RGBLED_GREEN: MSP1.P2.1/PM_UCA1CLK
- removed net P2.2_RGBLED_BLUE: MSP1.P2.2/PM_UCA1RXD/PM_UCA1SOMI
- removed net P2.3_IO_J4.34: MSP1.P2.3/PM_UCA1TXD/PM_UCA1SIMO
- removed net P3.0_IO_J2.18: MSP1.P3.0/PM_UCA2STE
- removed net P3.1_BCLUART_RTS: MSP1.P3.1/PM_UCA2CLK
- removed net P3.4_BCLUART_CTS: MSP1.P3.4/PM_UCB2STE
- removed net P3.5_IO_J4.32: MSP1.P3.5/PM_UCB2CLK
- removed net P3.6_IO_J2.11: MSP1.P3.6/PM_UCB2SIMO/PM_UCB2SDA
- removed net P3.7_IO_J4.31: MSP1.P3.7/PM_UCB2SOMI/PM_UCB2SCL
- removed net P4.0_A13_J3.24: MSP1.P4.0/A13
- removed net P4.1_IO_J1.5: MSP1.P4.1/A12
- removed net P4.2_A11_J3.25: MSP1.P4.2/ACLK/TA2CLK/A11
- removed net P4.3_A10_J1.6: MSP1.P4.3/MCLK/RTCCLK/A10
- removed net P4.4_A9_J3.26: MSP1.P4.4/HSMCLK/SVMHOUT/A9
- removed net P4.5_A8_J3.27: MSP1.P4.5/A8
- removed net P4.6_IO_J1.8: MSP1.P4.6/A7
- removed net P4.7_A6_J3.28: MSP1.P4.7/A6
- removed net P5.0_IO_J2.13: MSP1.P5.0/A5
- removed net P5.1_IO_J4.33: MSP1.P5.1/A4
- removed net P5.2_IO_J2.12: MSP1.P5.2/A3
- removed net P5.3: MSP1.P5.3/A2
Other:
- moved on the sheet: 12V_PDB, 5V_PDB

Commit message: PCB Updates
Connections:
- removed net N$1: MSP1.P9.1/A16
- removed net P10.0: MSP1.P10.0/UCB3STE
- removed net P10.1: MSP1.P10.1/UCB3CLK
- removed net P10.2: MSP1.P10.2/UCB3SIMO/UCB3SDA
- removed net P6.0_A15_J1.2: MSP1.P6.0/A15
- removed net P6.1_A14_J3.23: MSP1.P6.1/A14
- removed net P6.2: MSP1.P6.2/UCB1STE/C1.5
- removed net P6.3: MSP1.P6.3/UCB1CLK/C1.4
- removed net P6.4_I2CSDA_J1.10: MSP1.P6.4/UCB1SIMO/UCB1SDA/C1.3
- removed net P6.5_I2CSCL_J1.9: MSP1.P6.5/UCB1SOMI/UCB1SCL/C1.2
- removed net P7.0: MSP1.P7.0/PM_SMCLK/PM_DMAE0
- removed net P7.1: MSP1.P7.1/PM_C0OUT/PM_TA0CLK
- removed net P7.2: MSP1.P7.2/PM_C1OUT/PM_TA1CLK
- removed net P8.3: MSP1.P8.3/TA3CLK/A22
- removed net P8.4: MSP1.P8.4/A21
- removed net P8.5: MSP1.P8.5/A20
- removed net P8.6: MSP1.P8.6/A19
- removed net P8.7: MSP1.P8.7/A18
- removed net P9.0: MSP1.P9.0/A17
- removed net P9.4: MSP1.P9.4/UCA3STE
- removed net P9.5: MSP1.P9.5/UCA3CLK
- removed net P9.6: MSP1.P9.6/UCA3RXD/UCA3SOMI
- removed net P9.7: MSP1.P9.7/UCA3TXD/UCA3SIMO
Other:
- note added: "Flight Controller Interfacing"
- note added: "MCU <--> Motherboard Communication"
- note added: "Ultrasonic Sensors - Top and Bottom"
- note added: "Ultrasonic Sensors along Horizontal Plane"
- moved on the sheet: C14, C15, D1, L2, LEVEL_TRANSLATOR1, LEVEL_TRANSLATOR_2, LEVEL_TRANSLATOR_3, LM2596S, MOTHERBOARD_POWER_PINS, R4, R5, R6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

Commit message: Added Battery Monitroing Circuit
Parts:
- added BATTERY_MONITORING_PINS: (no value), pinhead:PINHD-2X3
- renumbered MOTHERBOPARD_TX to MOTHERBOARD_UART, MSP1 to MSP432P401R
Connections:
- new net P2.2_RX: BATTERY_MONITORING_PINS.1
- new net P3.6_SDA: BATTERY_MONITORING_PINS.3, MSP432P401R.P3.6/PM_UCB2SIMO/PM_UCB2SDA
- new net P3.7_SCL: BATTERY_MONITORING_PINS.4, MSP432P401R.P3.7/PM_UCB2SOMI/PM_UCB2SCL
- net 3V3: now also BATTERY_MONITORING_PINS.5
- net GND: now also BATTERY_MONITORING_PINS.2, BATTERY_MONITORING_PINS.6
Other:
- note added: "Battery Voltage Monitoring"
- note added: "Top and Bottom"
- note added: "Ultrasonic Sensors"
- note removed: "Ultrasonic Sensors - Top and Bottom"
- note removed: "VccA *must* be less than VccB!"
- moved on the sheet: ULTRA5

Commit message: Design Review PCB
Parts:
- removed C12, C13: 22p, rcl:C-EUCM0402
- removed C5, C6: 12p, rcl:C-EUCM0402
- removed IC2: LM317MB, v-reg:LM317MB
- removed Q1: 32.768kHz, microcrystal:MS3V-T1R
- removed Q2: KX-7 48MHz, Geyer:KX-7
- removed R1, R2: (no value), rcl:R-US_0204/5
- added U$2: TLV733P, texas:TLV733P
- BATTERY_MONITORING_PINS: device pinhead:PINHD-2X3 -> pinhead:PINHD-2X2
- C14, C15: device rcl:C-EUCM0402 -> eagle-ltspice:CC1206
- L2: device resistor:L-USL2012C -> resistor:L-USL3225M
Connections:
- removed net N$28: IC2.ADJ, R2.2
- removed net N$29: IC2.OUT, R1.2
- removed net N$7: C6.1, MSP432P401R.PJ.1/LFXOUT, Q1.1
- removed net N$8: C5.1, MSP432P401R.PJ.0/LFXIN, Q1.2
- removed net P10.5_V: ULTRA4.2
- removed net P5.2/XT2IN1: C13.1, MSP432P401R.PJ.3/HFXIN, Q2.2
- removed net P5.3/XT2OUT1: C12.1, MSP432P401R.PJ.2/HFXOUT, Q2.1
- net 12VDC: no longer C1.1, IC2.IN
- net 3V3: now also BATTERY_MONITORING_PINS.3; no longer BATTERY_MONITORING_PINS.5, R1.1
- net 5VDC: now also C1.1, U$2.EN_3, U$2.IN_1
- net GND: now also BATTERY_MONITORING_PINS.4, U$2.GND_2; no longer BATTERY_MONITORING_PINS.6, C12.2, C13.2, C5.2, C6.2, Q1.GND, R2.1
- net P10.5_5V: now also ULTRA4.2
- net P2.2_RX: now also MSP432P401R.P2.2/PM_UCA1RXD/PM_UCA1SOMI
- net P3.6_SDA: no longer BATTERY_MONITORING_PINS.3
- net P3.7_SCL: no longer BATTERY_MONITORING_PINS.4
Other:
- note removed: "HFX"
- note removed: "LFX"
- moved on the sheet: C1, C2, ULTRA4

Commit message: Completed Schematic for PCB submission
Parts:
- removed 12V_PDB, MOTHERBOARD_POWER_PINS: (no value), pinhead:PINHD-1X2
- removed C14: 680u, eagle-ltspice:CC1206
- removed C15: 220u, eagle-ltspice:CC1206
- removed D1: PD3S160, diode:PD3S160
- removed L2: 33u, resistor:L-USL3225M
- removed LM2596S: LM2596S, national-semiconductor:LM2596S
- added TP1, TP3: TPB1,27, testpad:TPB1,27
- added TP2: TPB2,54, testpad:TPB2,54
- C1, C2: device capacitor-wima:C2.5/2 -> rcl:C-EUC0805
- C11, C3, C4, C7, C8: device rcl:C-EUCM0402 -> rcl:C-EUC0805
- R4, R5, R6: value (none) -> 100k
- renumbered BATTERY_MONITORING_PINS to BATTERY_FC_PINS
Connections:
- removed net 12VDC: 12V_PDB.1, C14.1, LM2596S.VIN
- removed net MOTHEROARD_V+: C15.1, L2.2, LM2596S.FB, MOTHERBOARD_POWER_PINS.1
- removed net N$4: D1.C, L2.1, LM2596S.OUT
- removed net OE: R7.1, U$1.P$6
- net 3V3: now also R7.1, U$1.P$6
- net GND: now also TP2.TP; no longer 12V_PDB.2, C14.2, C15.2, D1.A, LM2596S.!ON!/OFF, LM2596S.GND, MOTHERBOARD_POWER_PINS.2
- net P2.2_RX: now also TP3.TP
- net P7.7: now also TP1.TP
- net P8.1: no longer LEVEL_TRANSLATOR1.A3
- net P8.2: now also LEVEL_TRANSLATOR1.A3
Other:
- note removed: "MotherBoard Power Circuit (5V,2.5A)"
- moved on the sheet: R7
